File: KiCad/Patchworks.kicad_sch (KiCad schematic)
At the start: 52 parts, among them J1 VEE Bolt, J10 5V Bus, J11 3V3 Bus, J12 DC, J2 VIN Bolt (4-40VDC), J3 GND Bolt, J4 3V3 Bus, J5 5V Bus, J6 5V Bus, J7 VCC Bus, J8 VCC Bus, J9 5V Bus, K1 Relay, M1 5V, Q1 2N3904, Q2 2N3904, SW1 Post, SW2 Power On, U1 LM317 Regulator (VCC 5-12VDC), U2 Power Monitor, U3 LCD Display, U4 BB Power, U5 PIC16F887-IP, Y1 4MHz

Commit message: Firmware and schematic updates
Parts:
- removed A2: Arduino Nano V3, Module:Arduino_Nano, symbol MCU_Module:Arduino_Nano_v3.x
- removed D4: Nano Act, symbol Device:LED
- removed D5: LED VCC, symbol Device:LED
- removed D6: PIC Act, symbol Device:LED
- removed R8: 1k, symbol Device:R_Small_US
- removed U5: PIC16F887-IP, symbol MCU_Microchip_PIC16:PIC16F887-IP
- removed Y1: 4MHz, symbol Device:Crystal
- added C6: 470uF, symbol Device:C_Polarized
- added D4: 1N4148, Diode_THT:D_DO-35_SOD27_P7.62mm_Horizontal, symbol Diode:1N4148
- added J13: External Clock, symbol Connector:Conn_01x01_Pin
- added J14: Breadboard Error, symbol Connector:Conn_01x01_Pin
- added J15: USB Power Out, symbol Connector:USB_A
- added Q3, Q4, Q5: 2N3904, Package_TO_SOT_THT:TO-92_Inline, symbol Transistor_BJT:2N3904
- added R10: 47K, symbol Device:R_Small_US
- added R11: 2K, symbol Device:R_Small_US
- added R12, R13, R18: 10K, symbol Device:R_Small_US
- added R14, R17: 1K, symbol Device:R_Small_US
- added R15, R16: 470R, symbol Device:R_Small_US
- added U5: ~, symbol Custom:Snubby Rev A 1.1
- C1, C2: value 47uF -> 470uF
- C3, C4: value 15pF -> 100nF
- F1: value 2A -> 1A
- J2: value VIN Bolt (4-40VDC) -> VIN Bolt (9-24VDC)
- R1: value 1k -> 470R
- R3: value 750R -> 47K
- R4: value 330R -> 2K
- R5: value 10k -> 47K
- R6: value 750R -> 2K
- U1: value LM317 Regulator (VCC 5-12VDC) -> LM317 Regulator (VCC 7-12VDC)
Connections:
- net GND: now also BT2.2 (-), C4.1, C5.1, J12.2, J3.1 (Pin_1), R4.2, C6.2, J15.4 (GND), J15.5 (Shield), Q3.1 (E), Q4.1 (E), R11.1, R12.1, R13.2, R15.2, R18.2, U5.6 (GND); no longer C4.2, C5.2, F1.1, J3.2 (Pin_2), Q2.1 (E)
- net at D1.1 (K), J10.1 (Pin_1), J5.4 (Pin_4)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: now also R1.2, D4.1 (K)
- net at D2.1 (K), M1.2 (-): now also D4.2 (A), Q5.3 (C); no longer Q1.3 (C)
- net at Q2.2 (B): now also R17.2, R18.1
- net at R5.1: now also A1.11 (A2), C4.2, R6.2
- net at J6.4 (Pin_4), J9.1 (Pin_1), R5.2: now also C6.1, J15.1 (VBUS), U5.3 (5V_RAIL_INPUT); no longer C5.1
- net at C3.1: now also A1.10 (A1), R3.2, R4.1
- net at Q1.2 (B): now also R14.2; no longer R1.2
- net at A1.24 (D9): now also R16.2; no longer R1.1
- net at C2.1, J11.1 (Pin_1), J4.4 (Pin_4): now also R10.2, U5.4 (3V3_RAIL_INPUT)
- net at K1.11, SW1.1: now also J3.2 (Pin_2); no longer F1.2
- net at C1.1, J7.4 (Pin_4), J8.1 (Pin_1)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: now also U5.1 (VCC), U5.2 (VCC_RAIL_INPUT)
- net at U1.1 (VIN): now also F1.1; no longer J2.2 (Pin_2)
- net at A1.21 (D6): now also R17.1
- net at A1.12 (A3): now also C5.2, R10.1, R11.2
- net at A1.25 (D10): now also J13.1 (Pin_1)
- net at A1.26 (D11): now also J14.1 (Pin_1)
- new net: Q1.3 (C), Q2.1 (E)
- new net: Q3.2 (B), R12.2, R15.1
- new net: Q3.3 (C), Q4.3 (C), Q5.1 (E)
- new net: R14.1, U5.5 (~{DETECT})
- new net: Q4.2 (B), R13.1, R16.1
- new net: Q5.2 (B), R1.1
- new net: F1.2, J2.2 (Pin_2)
- no-connect marks 85 -> 0
Other:
- note added: "3V3 Sense"
- note added: "5V Sense"
- note added: "Fan Breadboard Enable"
- note added: "Fan Breadboard Override"
- note added: "Fan Control"
- note added: "Fan MCU Enable"
- note added: "Relay Control"
- note added: "Relay MCU Enable"
- note added: "Snubby Enable"
- note added: "Squarely"
- note added: "VCC Sense"
- moved on the sheet: A1, BT1, BT2, BZ1, C2, D2, F1, Q2, R2, R9, TH1, U3

Commit message: Update Patchworks
Parts:
- removed BT2: Battery, symbol Device:Battery
- added F2: 1A, symbol Device:Fuse
- J1: value VEE Bolt -> VIN1 Bolt (9-24VDC)
- J10, J5, J6, J9: value 5V Bus -> VCC (3V3/5V) Bus
- J11, J4: value 3V3 Bus -> VCC (3V3/5V) Bus
- J2: value VIN Bolt (9-24VDC) -> VIN2 Bolt
- J7, J8: value VCC Bus -> VCC (VADJ) Bus
- U1: value LM317 Regulator (VCC 7-12VDC) -> LM317 Regulator (VADJ 7-12VDC)
Connections:
- net GND: now also BT1.2 (-)
- net at J1.2 (Pin_2): now also F1.1
- net at U1.1 (VIN): now also F1.2; no longer F1.1
- net at J2.2 (Pin_2): now also F2.1; no longer F1.2
- no-connect marks 0 -> 1
Other:
- moved on the sheet: BT1, F1
